File: sm83/alu_decoder.kicad_sch (KiCad schematic)
At the start: 11 parts

Commit message: SM83: Add data bus bridge schematic
Connections:
- new net: ALU_DECODER. (Y7), ALU_NOT5. (Y)
- new net: ALU_DECODER. (Y6), ALU_NOT4. (Y)
- new net: ALU_DECODER. (Y14), ALU_NOT10. (Y)
- new net: ALU_DECODER. (Y4), ALU_NOT2. (Y)
- new net: ALU_DECODER. (Y1), ALU_NOT1. (Y)
- new net: ALU_DECODER. (Y12), ALU_NOT9. (Y)
- new net: ALU_DECODER. (Y5), ALU_NOT3. (Y)
- new net: ALU_DECODER. (Y11), ALU_NOT8. (Y)
- new net: ALU_DECODER. (Y9), ALU_NOT6. (Y)
- new net: ALU_DECODER. (Y10), ALU_NOT7. (Y)

Commit message: Finish SM83 CPU schematic
Connections:
- new net: ALU_DECODER. (Y7), ALU_NOT5. (Y)
- new net: ALU_DECODER. (Y6), ALU_NOT4. (Y)
- new net: ALU_DECODER. (Y14), ALU_NOT10. (Y)
- new net: ALU_DECODER. (Y4), ALU_NOT2. (Y)
- new net: ALU_DECODER. (Y1), ALU_NOT1. (Y)
- new net: ALU_DECODER. (Y12), ALU_NOT9. (Y)
- new net: ALU_DECODER. (Y5), ALU_NOT3. (Y)
- new net: ALU_DECODER. (Y11), ALU_NOT8. (Y)
- new net: ALU_DECODER. (Y9), ALU_NOT6. (Y)
- new net: ALU_DECODER. (Y10), ALU_NOT7. (Y)
Changed lines of the file:
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@@
 	(title_block
 		(title "SM83 CPU")
-		(date "2025-12-08")
+		(date "2025-12-24")
 		(rev "0")
 		(company "CC-BY-SA-4.0 Michael Singer")

Commit message: SM83: Merge dist. NANDs and NOR from IRQ_PRIOs
Connections:
- new net: ALU_DECODER. (Y7), ALU_NOT5. (Y)
- new net: ALU_DECODER. (Y6), ALU_NOT4. (Y)
- new net: ALU_DECODER. (Y14), ALU_NOT10. (Y)
- new net: ALU_DECODER. (Y4), ALU_NOT2. (Y)
- new net: ALU_DECODER. (Y1), ALU_NOT1. (Y)
- new net: ALU_DECODER. (Y12), ALU_NOT9. (Y)
- new net: ALU_DECODER. (Y5), ALU_NOT3. (Y)
- new net: ALU_DECODER. (Y11), ALU_NOT8. (Y)
- new net: ALU_DECODER. (Y9), ALU_NOT6. (Y)
- new net: ALU_DECODER. (Y10), ALU_NOT7. (Y)
Changed lines of the file:
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@@
 	(title_block
 		(title "SM83 CPU")
-		(date "2025-12-24")
+		(date "2025-12-25")
 		(rev "0")
 		(company "CC-BY-SA-4.0 Michael Singer")

Commit message: Release version 0.9 of both schematics
Connections:
- new net: ALU_DECODER. (Y7), ALU_NOT5. (Y)
- new net: ALU_DECODER. (Y6), ALU_NOT4. (Y)
- new net: ALU_DECODER. (Y14), ALU_NOT10. (Y)
- new net: ALU_DECODER. (Y4), ALU_NOT2. (Y)
- new net: ALU_DECODER. (Y1), ALU_NOT1. (Y)
- new net: ALU_DECODER. (Y12), ALU_NOT9. (Y)
- new net: ALU_DECODER. (Y5), ALU_NOT3. (Y)
- new net: ALU_DECODER. (Y11), ALU_NOT8. (Y)
- new net: ALU_DECODER. (Y9), ALU_NOT6. (Y)
- new net: ALU_DECODER. (Y10), ALU_NOT7. (Y)
Changed lines of the file:
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@@
 		(title "SM83 CPU")
 		(date "2025-12-25")
-		(rev "0")
+		(rev "0.9")
 		(company "CC-BY-SA-4.0 Michael Singer")
 		(comment 1 "https://github.com/msinger/dmg-schematics")
