File: sm83/intr.kicad_sch (KiCad schematic)
At the start: 35 parts

Commit message: Finish SM83 CPU schematic
Connections:
- net at IRQ_PRIO1. (DIST_NOR_Y_N): now also IRQ_PRIO2. (DIST_NOR_Y_N); no longer IRQ_LATCH1. (~{Q})
- net at IRQ_PRIO5. (DIST_NOR_Y_N): now also IRQ_PRIO4. (DIST_NOR_Y_N); no longer IRQ_PRIO6. (DIST_NOR_Y_N)
- net at IRQ_PRIO4. (DIST_NOR_Y_N): now also IRQ_LATCH4. (~{Q}); no longer IRQ_PRIO5. (DIST_NOR_Y_N)
- net at IRQ_PRIO6. (DIST_NOR_Y_N): now also IRQ_PRIO7. (DIST_NOR_Y_N); no longer IRQ_LATCH6. (~{Q})
- net at IRQ_PRIO0. (DIST_NOR_Y_N): now also IRQ_LATCH0. (~{Q}); no longer IRQ_PRIO1. (DIST_NOR_Y_N)
- net at IRQ_PRIO2. (DIST_NOR_Y_N): now also IRQ_PRIO3. (DIST_NOR_Y_N); no longer IRQ_LATCH2. (~{Q})
- net at IRQ_PRIO3. (DIST_NOR_Y_N): now also IRQ_PRIO4. (DIST_NOR_Y_N); no longer IRQ_PRIO2. (DIST_NOR_Y_N)
- new net: IRQ_LATCH1. (~{Q}), IRQ_PRIO2. (AND_Y), IRQ_PRIO3. (AND_Y), IRQ_PRIO4. (AND_Y), IRQ_PRIO5. (AND_Y), IRQ_PRIO6. (AND_B_Y), IRQ_PRIO7. (DIST_NOR_Y_N)
- new net: IRQ_LATCH1. (~{Q}), IRQ_PRIO1. (DIST_NOR_Y_N)
- new net: IRQ_LATCH1. (~{Q}), IRQ_PRIO1. (AND_Y) (x2)
- new net: IRQ_LATCH1. (~{Q}), IRQ_NAND2_NAND3_1. (NAND_A_Y)
- new net: IRQ_PRIO5. (DIST_NOR_Y_N), IRQ_PRIO6. (DIST_NOR_Y_N)
- new net: IRQ_HEAD.1, IRQ_PRIO0. (DIST_NOR_Y_N), IRQ_PRIO1. (DIST_NOR_Y_N), IRQ_PRIO2. (DIST_NOR_Y_N), IRQ_PRIO3. (DIST_NOR_Y_N), IRQ_PRIO4. (DIST_NOR_Y_N), IRQ_PRIO5. (DIST_NOR_Y_N), IRQ_PRIO6. (DIST_NOR_Y_N), IRQ_PRIO7. (DIST_NOR_Y_N)
- new net: IRQ_LATCH5. (~{Q}), IRQ_PRIO5. (DIST_NOR_Y_N)
- new net: REG_IE0. (~{Q}), REG_IE1. (~{Q}), REG_IE2. (~{Q}), REG_IE3. (~{Q}), REG_IE4. (~{Q}), REG_IE5. (~{Q}), REG_IE6. (~{Q}), REG_IE7. (~{Q}), REG_IE_NOT_WE.2
- new net: IRQ_NAND2_NAND3_1. (NAND_B_Y), REG_IE1. (~{Q})
- new net: IRQ_NAND2_NAND3_1. (NAND_A_Y), REG_IE1. (~{Q})
- new net: IRQ_LATCH6. (~{Q}), IRQ_NAND2_NAND3_6. (NAND_A_Y)
- new net: IRQ_NAND2_NAND3_6. (NAND_A_Y), REG_IE6. (~{Q})
- new net: IRQ_LATCH6. (~{Q}), IRQ_PRIO6. (DIST_NOR_Y_N)
- new net: IRQ_NAND2_NAND3_0. (NAND_B_Y), REG_IE0. (~{Q})
- new net: IRQ_NAND2_NAND3_0. (NAND_A_Y), REG_IE0. (~{Q})
- new net: IRQ_HEAD.1, IRQ_PRIO0. (DIST_NAND_A_Y_N), IRQ_PRIO1. (DIST_NAND_A_Y_N), IRQ_PRIO2. (DIST_NAND_A_Y_N), IRQ_PRIO3. (DIST_NAND_A_Y_N), IRQ_PRIO4. (DIST_NAND_A_Y_N), IRQ_PRIO5. (DIST_NAND_A_Y_N), IRQ_PRIO6. (DIST_NAND_A_Y_N), IRQ_PRIO7. (DIST_NAND_A_Y_N)
- new net: IRQ_PRIO1. (DIST_NAND_A_Y_N), IRQ_PRIO2. (DIST_NAND_A_Y_N)
- new net: IRQ_PRIO2. (DIST_NAND_A_Y_N), IRQ_PRIO3. (DIST_NAND_A_Y_N)
- new net: IRQ_NAND2_NAND3_6. (NAND_B_Y), REG_IE6. (~{Q})
- new net: IRQ_PRIO0. (DIST_NAND_B_Y_N), IRQ_PRIO1. (DIST_NAND_B_Y_N)
- new net: IRQ_HEAD.1, IRQ_PRIO0. (DIST_NAND_B_Y_N), IRQ_PRIO1. (DIST_NAND_B_Y_N), IRQ_PRIO2. (DIST_NAND_B_Y_N), IRQ_PRIO3. (DIST_NAND_B_Y_N), IRQ_PRIO4. (DIST_NAND_B_Y_N), IRQ_PRIO5. (DIST_NAND_B_Y_N), IRQ_PRIO6. (DIST_NAND_B_Y_N), IRQ_PRIO7. (DIST_NAND_B_Y_N)
- new net: IRQ_LATCH2. (~{Q}), IRQ_NAND2_NAND3_2. (NAND_A_Y)
- new net: IRQ_NAND2_NAND3_2. (NAND_A_Y), REG_IE2. (~{Q})
- new net: IRQ_HEAD.2, IRQ_PRIO0. (AND_Y), IRQ_PRIO1. (AND_Y), IRQ_PRIO2. (AND_Y), IRQ_PRIO3. (AND_Y), IRQ_PRIO4. (AND_Y), IRQ_PRIO5. (AND_Y), IRQ_PRIO6. (AND_B_Y), IRQ_PRIO7. (DIST_NOR_Y_N)
- new net: IRQ_LATCH2. (~{Q}), IRQ_PRIO3. (AND_Y), IRQ_PRIO4. (AND_Y), IRQ_PRIO5. (AND_Y), IRQ_PRIO6. (AND_B_Y), IRQ_PRIO7. (DIST_NOR_Y_N)
- new net: IRQ_HEAD.1, IRQ_PRIO0. (AND_Y), IRQ_PRIO1. (AND_Y), IRQ_PRIO2. (AND_Y), IRQ_PRIO3. (AND_Y), IRQ_PRIO4. (AND_Y), IRQ_PRIO5. (AND_Y), IRQ_PRIO6. (AND_B_Y), IRQ_PRIO7. (DIST_NOR_Y_N)
- new net: IRQ_LATCH0. (~{Q}), IRQ_PRIO1. (AND_Y), IRQ_PRIO2. (AND_Y), IRQ_PRIO3. (AND_Y), IRQ_PRIO4. (AND_Y), IRQ_PRIO5. (AND_Y), IRQ_PRIO6. (AND_B_Y), IRQ_PRIO7. (DIST_NOR_Y_N)
- new net: IRQ_LATCH3. (~{Q}), IRQ_PRIO3. (AND_Y) (x2)
- new net: IRQ_PRIO1. (DIST_NAND_B_Y_N), IRQ_PRIO2. (DIST_NAND_B_Y_N)
- new net: IRQ_PRIO6. (DIST_NAND_B_Y_N), IRQ_PRIO7. (DIST_NAND_B_Y_N)
- new net: IRQ_PRIO5. (DIST_NAND_B_Y_N), IRQ_PRIO6. (DIST_NAND_B_Y_N)
- new net: IRQ_LATCH5. (~{Q}), IRQ_NAND2_NAND3_5. (NAND_A_Y)
- new net: IRQ_NAND2_NAND3_5. (NAND_A_Y), REG_IE5. (~{Q})
- new net: IRQ_LATCH6. (~{Q}), IRQ_PRIO6. (AND_B_Y) (x2)
- new net: IRQ_LATCH6. (~{Q}), IRQ_PRIO7. (DIST_NOR_Y_N)
- new net: IRQ_NAND2_NAND3_7. (NAND_A_Y), REG_IE7. (~{Q})
- new net: IRQ_LATCH7. (~{Q}), IRQ_NAND2_NAND3_7. (NAND_A_Y)
- new net: IRQ_PRIO0. (DIST_NAND_A_Y_N), IRQ_PRIO1. (DIST_NAND_A_Y_N)
- new net: IRQ_PRIO0. (DIST_NOR_Y_N), IRQ_PRIO1. (DIST_NOR_Y_N)
- new net: IRQ_LATCH5. (~{Q}), IRQ_PRIO6. (AND_B_Y), IRQ_PRIO7. (DIST_NOR_Y_N)
- new net: IRQ_LATCH5. (~{Q}), IRQ_PRIO5. (AND_Y) (x2)
- new net: IRQ_NAND2_NAND3_2. (NAND_B_Y), REG_IE2. (~{Q})
- new net: IRQ_LATCH2. (~{Q}), IRQ_PRIO2. (DIST_NOR_Y_N)
- new net: IRQ_LATCH3. (~{Q}), IRQ_PRIO4. (AND_Y), IRQ_PRIO5. (AND_Y), IRQ_PRIO6. (AND_B_Y), IRQ_PRIO7. (DIST_NOR_Y_N)
- new net: IRQ_LATCH4. (~{Q}), IRQ_PRIO5. (AND_Y), IRQ_PRIO6. (AND_B_Y), IRQ_PRIO7. (DIST_NOR_Y_N)
- new net: IRQ_NAND2_NAND3_5. (NAND_B_Y), REG_IE5. (~{Q})
- new net: IRQ_NAND2_NAND3_4. (NAND_A_Y), REG_IE4. (~{Q})
- new net: IRQ_LATCH4. (~{Q}), IRQ_NAND2_NAND3_4. (NAND_A_Y)
- new net: IRQ_NAND2_NAND3_3. (NAND_B_Y), REG_IE3. (~{Q})
- new net: IRQ_LATCH2. (~{Q}), IRQ_PRIO2. (AND_Y) (x2)
- new net: IRQ_NAND2_NAND3_7. (NAND_B_Y), REG_IE7. (~{Q})
- new net: IRQ_NAND2_NAND3_4. (NAND_B_Y), REG_IE4. (~{Q})
- new net: IRQ_LATCH3. (~{Q}), IRQ_NAND2_NAND3_3. (NAND_A_Y)
- new net: IRQ_NAND2_NAND3_3. (NAND_A_Y), REG_IE3. (~{Q})
- new net: IRQ_LATCH3. (~{Q}), IRQ_PRIO3. (DIST_NOR_Y_N)
- new net: IRQ_PRIO6. (DIST_NAND_A_Y_N), IRQ_PRIO7. (DIST_NAND_A_Y_N)
- new net: IRQ_PRIO5. (DIST_NAND_A_Y_N), IRQ_PRIO6. (DIST_NAND_A_Y_N)
- new net: IRQ_LATCH0. (~{Q}), IRQ_PRIO0. (AND_Y) (x2)
- new net: IRQ_PRIO3. (DIST_NAND_B_Y_N), IRQ_PRIO4. (DIST_NAND_B_Y_N)
- new net: IRQ_PRIO4. (DIST_NAND_B_Y_N), IRQ_PRIO5. (DIST_NAND_B_Y_N)
- new net: IRQ_LATCH7. (~{Q}), IRQ_PRIO7. (DIST_NOR_Y_N) (x3)
- new net: IRQ_PRIO2. (DIST_NAND_B_Y_N), IRQ_PRIO3. (DIST_NAND_B_Y_N)
- new net: IRQ_LATCH4. (~{Q}), IRQ_PRIO4. (AND_Y) (x2)
- new net: IRQ_LATCH0. (~{Q}), IRQ_NAND2_NAND3_0. (NAND_A_Y)
- new net: IRQ_PRIO3. (DIST_NAND_A_Y_N), IRQ_PRIO4. (DIST_NAND_A_Y_N)
- new net: IRQ_PRIO4. (DIST_NAND_A_Y_N), IRQ_PRIO5. (DIST_NAND_A_Y_N)
Changed lines of the file:
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@@
 	(title_block
 		(title "SM83 CPU")
-		(date "2025-12-08")
+		(date "2025-12-24")
 		(rev "0")
 		(company "CC-BY-SA-4.0 Michael Singer")

Commit message: SM83: Merge dist. NANDs and NOR from IRQ_PRIOs
Parts:
- removed unit 4 of IRQ_PRIO0
- removed unit 3 of IRQ_PRIO1
- removed unit 2 of IRQ_PRIO1
- removed unit 4 of IRQ_PRIO1
- removed unit 2 of IRQ_PRIO2
- removed unit 4 of IRQ_PRIO2
- removed unit 3 of IRQ_PRIO2
- removed unit 3 of IRQ_PRIO3
- removed unit 4 of IRQ_PRIO3
- removed unit 2 of IRQ_PRIO3
- removed unit 3 of IRQ_PRIO4
- removed unit 2 of IRQ_PRIO4
- removed unit 4 of IRQ_PRIO4
- removed unit 4 of IRQ_PRIO5
- removed unit 3 of IRQ_PRIO5
- removed unit 2 of IRQ_PRIO5
- removed unit 4 of IRQ_PRIO6
- removed unit 3 of IRQ_PRIO6
- removed unit 2 of IRQ_PRIO6
- removed unit 3 of IRQ_PRIO7
- removed unit 2 of IRQ_PRIO7
Connections:
- net A1: now also IRQ_PRIO0. (DIST_NAND_A_Y)
- net A10: now also IRQ_PRIO0. (DIST_NAND_B_Y)
- net A11: now also IRQ_PRIO0. (DIST_NAND_B_Y)
- net A12: now also IRQ_PRIO0. (DIST_NAND_B_Y)
- net A13: now also IRQ_PRIO0. (DIST_NAND_B_Y)
- net A14: now also IRQ_PRIO0. (DIST_NAND_B_Y)
- net A15: now also IRQ_PRIO0. (DIST_NAND_B_Y)
- net A2: now also IRQ_PRIO0. (DIST_NAND_A_Y)
- net A3: now also IRQ_PRIO0. (DIST_NAND_A_Y)
- net A4: now also IRQ_PRIO0. (DIST_NAND_A_Y)
- net A5: now also IRQ_PRIO0. (DIST_NAND_A_Y)
- net A6: now also IRQ_PRIO0. (DIST_NAND_A_Y)
- net A7: now also IRQ_PRIO0. (DIST_NAND_A_Y)
- net A9: now also IRQ_PRIO0. (DIST_NAND_B_Y)
- new net: IRQ_LATCH1. (~{Q}), IRQ_PRIO7. (DIST_NOR_Y)
- new net: IRQ_LATCH1. (~{Q}), IRQ_PRIO2. (AND_Y), IRQ_PRIO3. (AND_Y), IRQ_PRIO4. (AND_Y), IRQ_PRIO5. (AND_Y), IRQ_PRIO6. (AND_B_Y), IRQ_PRIO7. (DIST_NOR_Y)
- new net: IRQ_LATCH1. (~{Q}), IRQ_NAND2_NAND3_1. (NAND_A_Y)
- new net: IRQ_LATCH1. (~{Q}), IRQ_PRIO1. (AND_Y) (x2)
- new net: REG_IE0. (~{Q}), REG_IE1. (~{Q}), REG_IE2. (~{Q}), REG_IE3. (~{Q}), REG_IE4. (~{Q}), REG_IE5. (~{Q}), REG_IE6. (~{Q}), REG_IE7. (~{Q}), REG_IE_NOT_WE.2
- new net: IRQ_NAND2_NAND3_1. (NAND_B_Y), REG_IE1. (~{Q})
- new net: IRQ_NAND2_NAND3_1. (NAND_A_Y), REG_IE1. (~{Q})
- new net: IRQ_LATCH6. (~{Q}), IRQ_NAND2_NAND3_6. (NAND_A_Y)
- new net: IRQ_NAND2_NAND3_6. (NAND_A_Y), REG_IE6. (~{Q})
- new net: IRQ_NAND2_NAND3_0. (NAND_B_Y), REG_IE0. (~{Q})
- new net: IRQ_NAND2_NAND3_0. (NAND_A_Y), REG_IE0. (~{Q})
- new net: IRQ_NAND2_NAND3_6. (NAND_B_Y), REG_IE6. (~{Q})
- new net: IRQ_HEAD.2, IRQ_PRIO0. (AND_Y), IRQ_PRIO1. (AND_Y), IRQ_PRIO2. (AND_Y), IRQ_PRIO3. (AND_Y), IRQ_PRIO4. (AND_Y), IRQ_PRIO5. (AND_Y), IRQ_PRIO6. (AND_B_Y), IRQ_PRIO7. (DIST_NOR_Y)
- new net: IRQ_HEAD.1, IRQ_PRIO0. (AND_Y), IRQ_PRIO1. (AND_Y), IRQ_PRIO2. (AND_Y), IRQ_PRIO3. (AND_Y), IRQ_PRIO4. (AND_Y), IRQ_PRIO5. (AND_Y), IRQ_PRIO6. (AND_B_Y), IRQ_PRIO7. (DIST_NOR_Y)
- new net: IRQ_LATCH0. (~{Q}), IRQ_PRIO1. (AND_Y), IRQ_PRIO2. (AND_Y), IRQ_PRIO3. (AND_Y), IRQ_PRIO4. (AND_Y), IRQ_PRIO5. (AND_Y), IRQ_PRIO6. (AND_B_Y), IRQ_PRIO7. (DIST_NOR_Y)
- new net: IRQ_LATCH2. (~{Q}), IRQ_PRIO3. (AND_Y), IRQ_PRIO4. (AND_Y), IRQ_PRIO5. (AND_Y), IRQ_PRIO6. (AND_B_Y), IRQ_PRIO7. (DIST_NOR_Y)
- new net: IRQ_LATCH3. (~{Q}), IRQ_PRIO4. (AND_Y), IRQ_PRIO5. (AND_Y), IRQ_PRIO6. (AND_B_Y), IRQ_PRIO7. (DIST_NOR_Y)
- new net: IRQ_LATCH4. (~{Q}), IRQ_PRIO5. (AND_Y), IRQ_PRIO6. (AND_B_Y), IRQ_PRIO7. (DIST_NOR_Y)
- new net: IRQ_LATCH6. (~{Q}), IRQ_PRIO7. (DIST_NOR_Y) (x2)
- new net: IRQ_LATCH5. (~{Q}), IRQ_PRIO7. (DIST_NOR_Y)
- new net: IRQ_LATCH5. (~{Q}), IRQ_PRIO6. (AND_B_Y), IRQ_PRIO7. (DIST_NOR_Y)
- new net: IRQ_LATCH2. (~{Q}), IRQ_PRIO7. (DIST_NOR_Y)
- new net: IRQ_LATCH3. (~{Q}), IRQ_PRIO7. (DIST_NOR_Y)
- new net: IRQ_LATCH7. (~{Q}), IRQ_PRIO7. (DIST_NOR_Y) (x3)
- new net: IRQ_LATCH0. (~{Q}), IRQ_PRIO7. (DIST_NOR_Y)
- new net: IRQ_LATCH4. (~{Q}), IRQ_PRIO7. (DIST_NOR_Y)
- new net: IRQ_LATCH2. (~{Q}), IRQ_NAND2_NAND3_2. (NAND_A_Y)
- new net: IRQ_NAND2_NAND3_2. (NAND_A_Y), REG_IE2. (~{Q})
- new net: IRQ_LATCH0. (~{Q}), IRQ_PRIO0. (AND_Y) (x2)
- new net: IRQ_LATCH4. (~{Q}), IRQ_PRIO4. (AND_Y) (x2)
- new net: IRQ_LATCH5. (~{Q}), IRQ_PRIO5. (AND_Y) (x2)
- new net: IRQ_LATCH5. (~{Q}), IRQ_NAND2_NAND3_5. (NAND_A_Y)
- new net: IRQ_NAND2_NAND3_5. (NAND_A_Y), REG_IE5. (~{Q})
- new net: IRQ_LATCH6. (~{Q}), IRQ_PRIO6. (AND_B_Y) (x2)
- new net: IRQ_NAND2_NAND3_7. (NAND_A_Y), REG_IE7. (~{Q})
- new net: IRQ_LATCH7. (~{Q}), IRQ_NAND2_NAND3_7. (NAND_A_Y)
- new net: IRQ_LATCH3. (~{Q}), IRQ_PRIO3. (AND_Y) (x2)
- new net: IRQ_LATCH2. (~{Q}), IRQ_PRIO2. (AND_Y) (x2)
- new net: IRQ_NAND2_NAND3_2. (NAND_B_Y), REG_IE2. (~{Q})
- new net: IRQ_NAND2_NAND3_5. (NAND_B_Y), REG_IE5. (~{Q})
- new net: IRQ_NAND2_NAND3_4. (NAND_A_Y), REG_IE4. (~{Q})
- new net: IRQ_LATCH4. (~{Q}), IRQ_NAND2_NAND3_4. (NAND_A_Y)
- new net: IRQ_NAND2_NAND3_3. (NAND_B_Y), REG_IE3. (~{Q})
- new net: IRQ_NAND2_NAND3_7. (NAND_B_Y), REG_IE7. (~{Q})
- new net: IRQ_NAND2_NAND3_4. (NAND_B_Y), REG_IE4. (~{Q})
- new net: IRQ_LATCH3. (~{Q}), IRQ_NAND2_NAND3_3. (NAND_A_Y)
- new net: IRQ_NAND2_NAND3_3. (NAND_A_Y), REG_IE3. (~{Q})
- new net: IRQ_LATCH0. (~{Q}), IRQ_NAND2_NAND3_0. (NAND_A_Y)
Other:
- moved on the sheet: IRQ_HEADA, IRQ_HEADC, IRQ_HEADD

Commit message: Release version 0.9 of both schematics
Connections:
- new net: IRQ_LATCH1. (~{Q}), IRQ_PRIO7. (DIST_NOR_Y)
- new net: IRQ_LATCH1. (~{Q}), IRQ_PRIO2. (AND_Y), IRQ_PRIO3. (AND_Y), IRQ_PRIO4. (AND_Y), IRQ_PRIO5. (AND_Y), IRQ_PRIO6. (AND_B_Y), IRQ_PRIO7. (DIST_NOR_Y)
- new net: IRQ_LATCH1. (~{Q}), IRQ_NAND2_NAND3_1. (NAND_A_Y)
- new net: IRQ_LATCH1. (~{Q}), IRQ_PRIO1. (AND_Y) (x2)
- new net: REG_IE0. (~{Q}), REG_IE1. (~{Q}), REG_IE2. (~{Q}), REG_IE3. (~{Q}), REG_IE4. (~{Q}), REG_IE5. (~{Q}), REG_IE6. (~{Q}), REG_IE7. (~{Q}), REG_IE_NOT_WE.2
- new net: IRQ_NAND2_NAND3_1. (NAND_B_Y), REG_IE1. (~{Q})
- new net: IRQ_NAND2_NAND3_1. (NAND_A_Y), REG_IE1. (~{Q})
- new net: IRQ_LATCH6. (~{Q}), IRQ_NAND2_NAND3_6. (NAND_A_Y)
- new net: IRQ_NAND2_NAND3_6. (NAND_A_Y), REG_IE6. (~{Q})
- new net: IRQ_NAND2_NAND3_0. (NAND_B_Y), REG_IE0. (~{Q})
- new net: IRQ_NAND2_NAND3_0. (NAND_A_Y), REG_IE0. (~{Q})
- new net: IRQ_NAND2_NAND3_6. (NAND_B_Y), REG_IE6. (~{Q})
- new net: IRQ_HEAD.2, IRQ_PRIO0. (AND_Y), IRQ_PRIO1. (AND_Y), IRQ_PRIO2. (AND_Y), IRQ_PRIO3. (AND_Y), IRQ_PRIO4. (AND_Y), IRQ_PRIO5. (AND_Y), IRQ_PRIO6. (AND_B_Y), IRQ_PRIO7. (DIST_NOR_Y)
- new net: IRQ_HEAD.1, IRQ_PRIO0. (AND_Y), IRQ_PRIO1. (AND_Y), IRQ_PRIO2. (AND_Y), IRQ_PRIO3. (AND_Y), IRQ_PRIO4. (AND_Y), IRQ_PRIO5. (AND_Y), IRQ_PRIO6. (AND_B_Y), IRQ_PRIO7. (DIST_NOR_Y)
- new net: IRQ_LATCH0. (~{Q}), IRQ_PRIO1. (AND_Y), IRQ_PRIO2. (AND_Y), IRQ_PRIO3. (AND_Y), IRQ_PRIO4. (AND_Y), IRQ_PRIO5. (AND_Y), IRQ_PRIO6. (AND_B_Y), IRQ_PRIO7. (DIST_NOR_Y)
- new net: IRQ_LATCH2. (~{Q}), IRQ_PRIO3. (AND_Y), IRQ_PRIO4. (AND_Y), IRQ_PRIO5. (AND_Y), IRQ_PRIO6. (AND_B_Y), IRQ_PRIO7. (DIST_NOR_Y)
- new net: IRQ_LATCH3. (~{Q}), IRQ_PRIO4. (AND_Y), IRQ_PRIO5. (AND_Y), IRQ_PRIO6. (AND_B_Y), IRQ_PRIO7. (DIST_NOR_Y)
- new net: IRQ_LATCH4. (~{Q}), IRQ_PRIO5. (AND_Y), IRQ_PRIO6. (AND_B_Y), IRQ_PRIO7. (DIST_NOR_Y)
- new net: IRQ_LATCH6. (~{Q}), IRQ_PRIO7. (DIST_NOR_Y) (x2)
- new net: IRQ_LATCH5. (~{Q}), IRQ_PRIO7. (DIST_NOR_Y)
- new net: IRQ_LATCH5. (~{Q}), IRQ_PRIO6. (AND_B_Y), IRQ_PRIO7. (DIST_NOR_Y)
- new net: IRQ_LATCH2. (~{Q}), IRQ_PRIO7. (DIST_NOR_Y)
- new net: IRQ_LATCH3. (~{Q}), IRQ_PRIO7. (DIST_NOR_Y)
- new net: IRQ_LATCH7. (~{Q}), IRQ_PRIO7. (DIST_NOR_Y) (x3)
- new net: IRQ_LATCH0. (~{Q}), IRQ_PRIO7. (DIST_NOR_Y)
- new net: IRQ_LATCH4. (~{Q}), IRQ_PRIO7. (DIST_NOR_Y)
- new net: IRQ_LATCH2. (~{Q}), IRQ_NAND2_NAND3_2. (NAND_A_Y)
- new net: IRQ_NAND2_NAND3_2. (NAND_A_Y), REG_IE2. (~{Q})
- new net: IRQ_LATCH0. (~{Q}), IRQ_PRIO0. (AND_Y) (x2)
- new net: IRQ_LATCH4. (~{Q}), IRQ_PRIO4. (AND_Y) (x2)
- new net: IRQ_LATCH5. (~{Q}), IRQ_PRIO5. (AND_Y) (x2)
- new net: IRQ_LATCH5. (~{Q}), IRQ_NAND2_NAND3_5. (NAND_A_Y)
- new net: IRQ_NAND2_NAND3_5. (NAND_A_Y), REG_IE5. (~{Q})
- new net: IRQ_LATCH6. (~{Q}), IRQ_PRIO6. (AND_B_Y) (x2)
- new net: IRQ_NAND2_NAND3_7. (NAND_A_Y), REG_IE7. (~{Q})
- new net: IRQ_LATCH7. (~{Q}), IRQ_NAND2_NAND3_7. (NAND_A_Y)
- new net: IRQ_LATCH3. (~{Q}), IRQ_PRIO3. (AND_Y) (x2)
- new net: IRQ_LATCH2. (~{Q}), IRQ_PRIO2. (AND_Y) (x2)
- new net: IRQ_NAND2_NAND3_2. (NAND_B_Y), REG_IE2. (~{Q})
- new net: IRQ_NAND2_NAND3_5. (NAND_B_Y), REG_IE5. (~{Q})
- new net: IRQ_NAND2_NAND3_4. (NAND_A_Y), REG_IE4. (~{Q})
- new net: IRQ_LATCH4. (~{Q}), IRQ_NAND2_NAND3_4. (NAND_A_Y)
- new net: IRQ_NAND2_NAND3_3. (NAND_B_Y), REG_IE3. (~{Q})
- new net: IRQ_NAND2_NAND3_7. (NAND_B_Y), REG_IE7. (~{Q})
- new net: IRQ_NAND2_NAND3_4. (NAND_B_Y), REG_IE4. (~{Q})
- new net: IRQ_LATCH3. (~{Q}), IRQ_NAND2_NAND3_3. (NAND_A_Y)
- new net: IRQ_NAND2_NAND3_3. (NAND_A_Y), REG_IE3. (~{Q})
- new net: IRQ_LATCH0. (~{Q}), IRQ_NAND2_NAND3_0. (NAND_A_Y)
Changed lines of the file:
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@@
 		(title "SM83 CPU")
 		(date "2025-12-25")
-		(rev "0")
+		(rev "0.9")
 		(company "CC-BY-SA-4.0 Michael Singer")
 		(comment 1 "https://github.com/msinger/dmg-schematics")

Commit message: Release revision 0.10 of both schematics
Connections:
- new net: IRQ_LATCH1. (~{Q}), IRQ_PRIO7. (DIST_NOR_Y)
- new net: IRQ_LATCH1. (~{Q}), IRQ_PRIO2. (AND_Y), IRQ_PRIO3. (AND_Y), IRQ_PRIO4. (AND_Y), IRQ_PRIO5. (AND_Y), IRQ_PRIO6. (AND_B_Y), IRQ_PRIO7. (DIST_NOR_Y)
- new net: IRQ_LATCH1. (~{Q}), IRQ_NAND2_NAND3_1. (NAND_A_Y)
- new net: IRQ_LATCH1. (~{Q}), IRQ_PRIO1. (AND_Y) (x2)
- new net: REG_IE0. (~{Q}), REG_IE1. (~{Q}), REG_IE2. (~{Q}), REG_IE3. (~{Q}), REG_IE4. (~{Q}), REG_IE5. (~{Q}), REG_IE6. (~{Q}), REG_IE7. (~{Q}), REG_IE_NOT_WE.2
- new net: IRQ_NAND2_NAND3_1. (NAND_B_Y), REG_IE1. (~{Q})
- new net: IRQ_NAND2_NAND3_1. (NAND_A_Y), REG_IE1. (~{Q})
- new net: IRQ_LATCH6. (~{Q}), IRQ_NAND2_NAND3_6. (NAND_A_Y)
- new net: IRQ_NAND2_NAND3_6. (NAND_A_Y), REG_IE6. (~{Q})
- new net: IRQ_NAND2_NAND3_0. (NAND_B_Y), REG_IE0. (~{Q})
- new net: IRQ_NAND2_NAND3_0. (NAND_A_Y), REG_IE0. (~{Q})
- new net: IRQ_NAND2_NAND3_6. (NAND_B_Y), REG_IE6. (~{Q})
- new net: IRQ_HEAD.2, IRQ_PRIO0. (AND_Y), IRQ_PRIO1. (AND_Y), IRQ_PRIO2. (AND_Y), IRQ_PRIO3. (AND_Y), IRQ_PRIO4. (AND_Y), IRQ_PRIO5. (AND_Y), IRQ_PRIO6. (AND_B_Y), IRQ_PRIO7. (DIST_NOR_Y)
- new net: IRQ_HEAD.1, IRQ_PRIO0. (AND_Y), IRQ_PRIO1. (AND_Y), IRQ_PRIO2. (AND_Y), IRQ_PRIO3. (AND_Y), IRQ_PRIO4. (AND_Y), IRQ_PRIO5. (AND_Y), IRQ_PRIO6. (AND_B_Y), IRQ_PRIO7. (DIST_NOR_Y)
- new net: IRQ_LATCH0. (~{Q}), IRQ_PRIO1. (AND_Y), IRQ_PRIO2. (AND_Y), IRQ_PRIO3. (AND_Y), IRQ_PRIO4. (AND_Y), IRQ_PRIO5. (AND_Y), IRQ_PRIO6. (AND_B_Y), IRQ_PRIO7. (DIST_NOR_Y)
- new net: IRQ_LATCH2. (~{Q}), IRQ_PRIO3. (AND_Y), IRQ_PRIO4. (AND_Y), IRQ_PRIO5. (AND_Y), IRQ_PRIO6. (AND_B_Y), IRQ_PRIO7. (DIST_NOR_Y)
- new net: IRQ_LATCH3. (~{Q}), IRQ_PRIO4. (AND_Y), IRQ_PRIO5. (AND_Y), IRQ_PRIO6. (AND_B_Y), IRQ_PRIO7. (DIST_NOR_Y)
- new net: IRQ_LATCH4. (~{Q}), IRQ_PRIO5. (AND_Y), IRQ_PRIO6. (AND_B_Y), IRQ_PRIO7. (DIST_NOR_Y)
- new net: IRQ_LATCH6. (~{Q}), IRQ_PRIO7. (DIST_NOR_Y) (x2)
- new net: IRQ_LATCH5. (~{Q}), IRQ_PRIO7. (DIST_NOR_Y)
- new net: IRQ_LATCH5. (~{Q}), IRQ_PRIO6. (AND_B_Y), IRQ_PRIO7. (DIST_NOR_Y)
- new net: IRQ_LATCH2. (~{Q}), IRQ_PRIO7. (DIST_NOR_Y)
- new net: IRQ_LATCH3. (~{Q}), IRQ_PRIO7. (DIST_NOR_Y)
- new net: IRQ_LATCH7. (~{Q}), IRQ_PRIO7. (DIST_NOR_Y) (x3)
- new net: IRQ_LATCH0. (~{Q}), IRQ_PRIO7. (DIST_NOR_Y)
- new net: IRQ_LATCH4. (~{Q}), IRQ_PRIO7. (DIST_NOR_Y)
- new net: IRQ_LATCH2. (~{Q}), IRQ_NAND2_NAND3_2. (NAND_A_Y)
- new net: IRQ_NAND2_NAND3_2. (NAND_A_Y), REG_IE2. (~{Q})
- new net: IRQ_LATCH0. (~{Q}), IRQ_PRIO0. (AND_Y) (x2)
- new net: IRQ_LATCH4. (~{Q}), IRQ_PRIO4. (AND_Y) (x2)
- new net: IRQ_LATCH5. (~{Q}), IRQ_PRIO5. (AND_Y) (x2)
- new net: IRQ_LATCH5. (~{Q}), IRQ_NAND2_NAND3_5. (NAND_A_Y)
- new net: IRQ_NAND2_NAND3_5. (NAND_A_Y), REG_IE5. (~{Q})
- new net: IRQ_LATCH6. (~{Q}), IRQ_PRIO6. (AND_B_Y) (x2)
- new net: IRQ_NAND2_NAND3_7. (NAND_A_Y), REG_IE7. (~{Q})
- new net: IRQ_LATCH7. (~{Q}), IRQ_NAND2_NAND3_7. (NAND_A_Y)
- new net: IRQ_LATCH3. (~{Q}), IRQ_PRIO3. (AND_Y) (x2)
- new net: IRQ_LATCH2. (~{Q}), IRQ_PRIO2. (AND_Y) (x2)
- new net: IRQ_NAND2_NAND3_2. (NAND_B_Y), REG_IE2. (~{Q})
- new net: IRQ_NAND2_NAND3_5. (NAND_B_Y), REG_IE5. (~{Q})
- new net: IRQ_NAND2_NAND3_4. (NAND_A_Y), REG_IE4. (~{Q})
- new net: IRQ_LATCH4. (~{Q}), IRQ_NAND2_NAND3_4. (NAND_A_Y)
- new net: IRQ_NAND2_NAND3_3. (NAND_B_Y), REG_IE3. (~{Q})
- new net: IRQ_NAND2_NAND3_7. (NAND_B_Y), REG_IE7. (~{Q})
- new net: IRQ_NAND2_NAND3_4. (NAND_B_Y), REG_IE4. (~{Q})
- new net: IRQ_LATCH3. (~{Q}), IRQ_NAND2_NAND3_3. (NAND_A_Y)
- new net: IRQ_NAND2_NAND3_3. (NAND_A_Y), REG_IE3. (~{Q})
- new net: IRQ_LATCH0. (~{Q}), IRQ_NAND2_NAND3_0. (NAND_A_Y)
Changed lines of the file:
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@@
 	(title_block
 		(title "SM83 CPU")
-		(date "2025-12-25")
-		(rev "0.9")
+		(date "2026-03-22")
+		(rev "0.10")
 		(company "CC-BY-SA-4.0 Michael Singer")
 		(comment 1 "https://github.com/msinger/dmg-schematics")
@@
 		)
 		(instances
-			(project ""
+			(project "sm83"
 				(path "/8717d046-1dfd-46fe-a5f7-4e4d2f07de68/1b42a619-7459-4edd-bc6f-370029071d58"
 					(reference "REG_IE0")
@@
 		)
 		(instances
-			(project ""
+			(project "sm83"
 				(path "/8717d046-1dfd-46fe-a5f7-4e4d2f07de68/1b42a619-7459-4edd-bc6f-370029071d58"
 					(reference "REG_IE_NOT_WE")
@@
 		)
 		(instances
-			(project ""
+			(project "sm83"
 				(path "/8717d046-1dfd-46fe-a5f7-4e4d2f07de68/1b42a619-7459-4edd-bc6f-370029071d58"
 					(reference "IRQ_PRIO7")
@@
 		)
 		(instances
-			(project ""
+			(project "sm83"
 				(path "/8717d046-1dfd-46fe-a5f7-4e4d2f07de68/1b42a619-7459-4edd-bc6f-370029071d58"
 					(reference "IRQ_PRIO0")
@@
 		)
 		(instances
-			(project ""
+			(project "sm83"
 				(path "/8717d046-1dfd-46fe-a5f7-4e4d2f07de68/1b42a619-7459-4edd-bc6f-370029071d58"
 					(reference "IRQ_PRIO4")
@@
 		)
 		(instances
-			(project ""
+			(project "sm83"
 				(path "/8717d046-1dfd-46fe-a5f7-4e4d2f07de68/1b42a619-7459-4edd-bc6f-370029071d58"
 					(reference "IRQ_HEAD")
@@
 		)
 		(instances
-			(project ""
+			(project "sm83"
 				(path "/8717d046-1dfd-46fe-a5f7-4e4d2f07de68/1b42a619-7459-4edd-bc6f-370029071d58"
 					(reference "IRQ_PRIO5")
@@
 		)
 		(instances
-			(project ""
+			(project "sm83"
 				(path "/8717d046-1dfd-46fe-a5f7-4e4d2f07de68/1b42a619-7459-4edd-bc6f-370029071d58"
 					(reference "IRQ_HEAD")
@@
 		)
 		(instances
-			(project ""
+			(project "sm83"
 				(path "/8717d046-1dfd-46fe-a5f7-4e4d2f07de68/1b42a619-7459-4edd-bc6f-370029071d58"
 					(reference "IRQ_NAND2_NAND3_0")
@@
 		)
 		(instances
-			(project ""
+			(project "sm83"
 				(path "/8717d046-1dfd-46fe-a5f7-4e4d2f07de68/1b42a619-7459-4edd-bc6f-370029071d58"
 					(reference "IRQ_PRIO3")
@@
 		)
 		(instances
-			(project ""
+			(project "sm83"
 				(path "/8717d046-1dfd-46fe-a5f7-4e4d2f07de68/1b42a619-7459-4edd-bc6f-370029071d58"
 					(reference "IRQ_AND")
@@
 		)
 		(instances
-			(project ""
+			(project "sm83"
 				(path "/8717d046-1dfd-46fe-a5f7-4e4d2f07de68/1b42a619-7459-4edd-bc6f-370029071d58"
 					(reference "IRQ_PRIO2")
@@
 		)
 		(instances
-			(project ""
+			(project "sm83"
 				(path "/8717d046-1dfd-46fe-a5f7-4e4d2f07de68/1b42a619-7459-4edd-bc6f-370029071d58"
 					(reference "IRQ_HEAD")
@@
 		)
 		(instances
-			(project ""
+			(project "sm83"
 				(path "/8717d046-1dfd-46fe-a5f7-4e4d2f07de68/1b42a619-7459-4edd-bc6f-370029071d58"
 					(reference "IRQ_PRIO0")
@@
 		)
 		(instances
-			(project ""
+			(project "sm83"
 				(path "/8717d046-1dfd-46fe-a5f7-4e4d2f07de68/1b42a619-7459-4edd-bc6f-370029071d58"
 					(reference "IRQ_PRIO0")
@@
 		)
 		(instances
-			(project ""
+			(project "sm83"
 				(path "/8717d046-1dfd-46fe-a5f7-4e4d2f07de68/1b42a619-7459-4edd-bc6f-370029071d58"
 					(reference "IRQ_NAND2_NAND3_0")
@@
 		)
 		(instances
-			(project ""
+			(project "sm83"
 				(path "/8717d046-1dfd-46fe-a5f7-4e4d2f07de68/1b42a619-7459-4edd-bc6f-370029071d58"
 					(reference "IRQ_HEAD")
@@
 		)
 		(instances
-			(project ""
+			(project "sm83"
 				(path "/8717d046-1dfd-46fe-a5f7-4e4d2f07de68/1b42a619-7459-4edd-bc6f-370029071d58"
 					(reference "IRQ_LATCH0")
@@
 		)
 		(instances
-			(project ""
+			(project "sm83"
 				(path "/8717d046-1dfd-46fe-a5f7-4e4d2f07de68/1b42a619-7459-4edd-bc6f-370029071d58"
 					(reference "IRQ_PRIO6")
@@
 		)
 		(instances
-			(project ""
+			(project "sm83"
 				(path "/8717d046-1dfd-46fe-a5f7-4e4d2f07de68/1b42a619-7459-4edd-bc6f-370029071d58"
 					(reference "IRQ_HEAD")
@@
 		)
 		(instances
-			(project ""
+			(project "sm83"
 				(path "/8717d046-1dfd-46fe-a5f7-4e4d2f07de68/1b42a619-7459-4edd-bc6f-370029071d58"
 					(reference "IRQ_PRIO1")
