File: sm83/intr.kicad_sch (KiCad schematic)
At the start: 35 parts

Commit message: Release revision 0.11 of both schematics
Connections:
- new net: IRQ_LATCH1. (~{Q}), IRQ_PRIO7. (DIST_NOR_Y)
- new net: IRQ_LATCH1. (~{Q}), IRQ_PRIO2. (AND_Y), IRQ_PRIO3. (AND_Y), IRQ_PRIO4. (AND_Y), IRQ_PRIO5. (AND_Y), IRQ_PRIO6. (AND_B_Y), IRQ_PRIO7. (DIST_NOR_Y)
- new net: IRQ_LATCH1. (~{Q}), IRQ_NAND2_NAND3_1. (NAND_A_Y)
- new net: IRQ_LATCH1. (~{Q}), IRQ_PRIO1. (AND_Y) (x2)
- new net: REG_IE0. (~{Q}), REG_IE1. (~{Q}), REG_IE2. (~{Q}), REG_IE3. (~{Q}), REG_IE4. (~{Q}), REG_IE5. (~{Q}), REG_IE6. (~{Q}), REG_IE7. (~{Q}), REG_IE_NOT_WE.2
- new net: IRQ_NAND2_NAND3_1. (NAND_B_Y), REG_IE1. (~{Q})
- new net: IRQ_NAND2_NAND3_1. (NAND_A_Y), REG_IE1. (~{Q})
- new net: IRQ_LATCH6. (~{Q}), IRQ_NAND2_NAND3_6. (NAND_A_Y)
- new net: IRQ_NAND2_NAND3_6. (NAND_A_Y), REG_IE6. (~{Q})
- new net: IRQ_NAND2_NAND3_0. (NAND_B_Y), REG_IE0. (~{Q})
- new net: IRQ_NAND2_NAND3_0. (NAND_A_Y), REG_IE0. (~{Q})
- new net: IRQ_NAND2_NAND3_6. (NAND_B_Y), REG_IE6. (~{Q})
- new net: IRQ_HEAD.2, IRQ_PRIO0. (AND_Y), IRQ_PRIO1. (AND_Y), IRQ_PRIO2. (AND_Y), IRQ_PRIO3. (AND_Y), IRQ_PRIO4. (AND_Y), IRQ_PRIO5. (AND_Y), IRQ_PRIO6. (AND_B_Y), IRQ_PRIO7. (DIST_NOR_Y)
- new net: IRQ_HEAD.1, IRQ_PRIO0. (AND_Y), IRQ_PRIO1. (AND_Y), IRQ_PRIO2. (AND_Y), IRQ_PRIO3. (AND_Y), IRQ_PRIO4. (AND_Y), IRQ_PRIO5. (AND_Y), IRQ_PRIO6. (AND_B_Y), IRQ_PRIO7. (DIST_NOR_Y)
- new net: IRQ_LATCH0. (~{Q}), IRQ_PRIO1. (AND_Y), IRQ_PRIO2. (AND_Y), IRQ_PRIO3. (AND_Y), IRQ_PRIO4. (AND_Y), IRQ_PRIO5. (AND_Y), IRQ_PRIO6. (AND_B_Y), IRQ_PRIO7. (DIST_NOR_Y)
- new net: IRQ_LATCH2. (~{Q}), IRQ_PRIO3. (AND_Y), IRQ_PRIO4. (AND_Y), IRQ_PRIO5. (AND_Y), IRQ_PRIO6. (AND_B_Y), IRQ_PRIO7. (DIST_NOR_Y)
- new net: IRQ_LATCH3. (~{Q}), IRQ_PRIO4. (AND_Y), IRQ_PRIO5. (AND_Y), IRQ_PRIO6. (AND_B_Y), IRQ_PRIO7. (DIST_NOR_Y)
- new net: IRQ_LATCH4. (~{Q}), IRQ_PRIO5. (AND_Y), IRQ_PRIO6. (AND_B_Y), IRQ_PRIO7. (DIST_NOR_Y)
- new net: IRQ_LATCH6. (~{Q}), IRQ_PRIO7. (DIST_NOR_Y) (x2)
- new net: IRQ_LATCH5. (~{Q}), IRQ_PRIO7. (DIST_NOR_Y)
- new net: IRQ_LATCH5. (~{Q}), IRQ_PRIO6. (AND_B_Y), IRQ_PRIO7. (DIST_NOR_Y)
- new net: IRQ_LATCH2. (~{Q}), IRQ_PRIO7. (DIST_NOR_Y)
- new net: IRQ_LATCH3. (~{Q}), IRQ_PRIO7. (DIST_NOR_Y)
- new net: IRQ_LATCH7. (~{Q}), IRQ_PRIO7. (DIST_NOR_Y) (x3)
- new net: IRQ_LATCH0. (~{Q}), IRQ_PRIO7. (DIST_NOR_Y)
- new net: IRQ_LATCH4. (~{Q}), IRQ_PRIO7. (DIST_NOR_Y)
- new net: IRQ_LATCH2. (~{Q}), IRQ_NAND2_NAND3_2. (NAND_A_Y)
- new net: IRQ_NAND2_NAND3_2. (NAND_A_Y), REG_IE2. (~{Q})
- new net: IRQ_LATCH0. (~{Q}), IRQ_PRIO0. (AND_Y) (x2)
- new net: IRQ_LATCH4. (~{Q}), IRQ_PRIO4. (AND_Y) (x2)
- new net: IRQ_LATCH5. (~{Q}), IRQ_PRIO5. (AND_Y) (x2)
- new net: IRQ_LATCH5. (~{Q}), IRQ_NAND2_NAND3_5. (NAND_A_Y)
- new net: IRQ_NAND2_NAND3_5. (NAND_A_Y), REG_IE5. (~{Q})
- new net: IRQ_LATCH6. (~{Q}), IRQ_PRIO6. (AND_B_Y) (x2)
- new net: IRQ_NAND2_NAND3_7. (NAND_A_Y), REG_IE7. (~{Q})
- new net: IRQ_LATCH7. (~{Q}), IRQ_NAND2_NAND3_7. (NAND_A_Y)
- new net: IRQ_LATCH3. (~{Q}), IRQ_PRIO3. (AND_Y) (x2)
- new net: IRQ_LATCH2. (~{Q}), IRQ_PRIO2. (AND_Y) (x2)
- new net: IRQ_NAND2_NAND3_2. (NAND_B_Y), REG_IE2. (~{Q})
- new net: IRQ_NAND2_NAND3_5. (NAND_B_Y), REG_IE5. (~{Q})
- new net: IRQ_NAND2_NAND3_4. (NAND_A_Y), REG_IE4. (~{Q})
- new net: IRQ_LATCH4. (~{Q}), IRQ_NAND2_NAND3_4. (NAND_A_Y)
- new net: IRQ_NAND2_NAND3_3. (NAND_B_Y), REG_IE3. (~{Q})
- new net: IRQ_NAND2_NAND3_7. (NAND_B_Y), REG_IE7. (~{Q})
- new net: IRQ_NAND2_NAND3_4. (NAND_B_Y), REG_IE4. (~{Q})
- new net: IRQ_LATCH3. (~{Q}), IRQ_NAND2_NAND3_3. (NAND_A_Y)
- new net: IRQ_NAND2_NAND3_3. (NAND_A_Y), REG_IE3. (~{Q})
- new net: IRQ_LATCH0. (~{Q}), IRQ_NAND2_NAND3_0. (NAND_A_Y)
Changed lines of the file:
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@@
 	(title_block
 		(title "SM83 CPU")
-		(date "2026-03-22")
-		(rev "0.10")
+		(date "2026-04-11")
+		(rev "0.11")
 		(company "CC-BY-SA-4.0 Michael Singer")
 		(comment 1 "https://github.com/msinger/dmg-schematics")
