File: sm83/reg_gp.kicad_sch (KiCad schematic)
At the start: 117 parts

Commit message: Release revision 0.11 of both schematics
Connections:
- new net: REG_B2. (Q), REG_BC_OUT2. (C_Y1)
- new net: REG_BC_OUT2. (C_Y1), REG_C2. (Q)
- new net: REG_L0. (Q), REG_L1. (Q), REG_L2. (Q), REG_L3. (Q), REG_L4. (Q), REG_L5. (Q), REG_L6. (Q), REG_L7. (Q), REG_L_NOT_WE.2
- new net: REG_HL_OUT1. (L_Y1), REG_L1. (Q)
- new net: REG_D0. (Q), REG_D1. (Q), REG_D2. (Q), REG_D3. (Q), REG_D4. (Q), REG_D5. (Q), REG_D6. (Q), REG_D7. (Q), REG_D_NOT_WE.2
- new net: REG_D2. (Q), REG_DE_OUT2. (D_Y1)
- new net: REG_HL_OUT0. (L_Y1), REG_L0. (Q)
- new net: REG_IR0. (Q), REG_IR1. (Q), REG_IR2. (Q), REG_IR3. (Q), REG_IR4. (Q), REG_IR5. (Q), REG_IR6. (Q), REG_IR7. (Q), REG_IR_NOT_WE.2
- new net: REG_B0. (Q), REG_B1. (Q), REG_B2. (Q), REG_B3. (Q), REG_B4. (Q), REG_B5. (Q), REG_B6. (Q), REG_B7. (Q), REG_B_NOT_WE.2
- new net: REG_B6. (Q), REG_BC_OUT6. (C_Y1)
- new net: REG_A2. (Q), REG_A_OUT2. (B_Y), REG_OA1.2
- new net: REG_H0. (Q), REG_H1. (Q), REG_H2. (Q), REG_H3. (Q), REG_H4. (Q), REG_H5. (Q), REG_H6. (Q), REG_H7. (Q), REG_H_NOT_WE.2
- new net: REG_H1. (Q), REG_HL_OUT1. (L_Y1)
- new net: REG_A0. (Q), REG_A1. (Q), REG_A2. (Q), REG_A3. (Q), REG_A4. (Q), REG_A5. (Q), REG_A6. (Q), REG_A7. (Q), REG_A_NOT_WE.2
- new net: REG_A5. (Q), REG_A_OUT5. (B_Y), REG_OA2.1
- new net: REG_HL_OUT3. (L_Y1), REG_L3. (Q)
- new net: REG_B4. (Q), REG_BC_OUT4. (C_Y1)
- new net: REG_E0. (Q), REG_E1. (Q), REG_E2. (Q), REG_E3. (Q), REG_E4. (Q), REG_E5. (Q), REG_E6. (Q), REG_E7. (Q), REG_E_NOT_WE.2
- new net: REG_DE_OUT0. (D_Y1), REG_E0. (Q)
- new net: REG_DE_OUT7. (D_Y1), REG_E7. (Q)
- new net: REG_C0. (Q), REG_C1. (Q), REG_C2. (Q), REG_C3. (Q), REG_C4. (Q), REG_C5. (Q), REG_C6. (Q), REG_C7. (Q), REG_C_NOT_WE.2
- new net: REG_H4. (Q), REG_HL_OUT4. (L_Y1)
- new net: REG_HL_OUT7. (L_Y1), REG_L7. (Q)
- new net: REG_D5. (Q), REG_DE_OUT5. (D_Y1)
- new net: REG_DE_OUT5. (D_Y1), REG_E5. (Q)
- new net: REG_HL_OUT4. (L_Y1), REG_L4. (Q)
- new net: REG_A3. (Q), REG_A_OUT3. (B_Y), REG_OA1.3
- new net: REG_D7. (Q), REG_DE_OUT7. (D_Y1)
- new net: REG_B0. (Q), REG_BC_OUT0. (C_Y1)
- new net: REG_BC_OUT0. (C_Y1), REG_C0. (Q)
- new net: REG_D1. (Q), REG_DE_OUT1. (D_Y1)
- new net: REG_DE_OUT6. (D_Y1), REG_E6. (Q)
- new net: REG_HL_OUT2. (L_Y1), REG_L2. (Q)
- new net: REG_BC_OUT4. (C_Y1), REG_C4. (Q)
- new net: REG_DE_OUT4. (D_Y1), REG_E4. (Q)
- new net: REG_D4. (Q), REG_DE_OUT4. (D_Y1)
- new net: REG_DE_OUT3. (D_Y1), REG_E3. (Q)
- new net: REG_D3. (Q), REG_DE_OUT3. (D_Y1)
- new net: REG_H3. (Q), REG_HL_OUT3. (L_Y1)
- new net: REG_B1. (Q), REG_BC_OUT1. (C_Y1)
- new net: REG_H6. (Q), REG_HL_OUT6. (L_Y1)
- new net: REG_BC_OUT7. (C_Y1), REG_C7. (Q)
- new net: REG_B7. (Q), REG_BC_OUT7. (C_Y1)
- new net: REG_A4. (Q), REG_AND.2, REG_A_OUT4. (B_Y)
- new net: REG_A1. (Q), REG_A_OUT1. (B_Y), REG_OA1.1
- new net: REG_H7. (Q), REG_HL_OUT7. (L_Y1)
- new net: REG_H0. (Q), REG_HL_OUT0. (L_Y1)
- new net: REG_A6. (Q), REG_A_OUT6. (B_Y), REG_OA2.2
- new net: REG_H2. (Q), REG_HL_OUT2. (L_Y1)
- new net: REG_BC_OUT6. (C_Y1), REG_C6. (Q)
- new net: REG_D0. (Q), REG_DE_OUT0. (D_Y1)
- new net: REG_DE_OUT2. (D_Y1), REG_E2. (Q)
- new net: REG_D6. (Q), REG_DE_OUT6. (D_Y1)
- new net: REG_BC_OUT3. (C_Y1), REG_C3. (Q)
- new net: REG_BC_OUT5. (C_Y1), REG_C5. (Q)
- new net: REG_B5. (Q), REG_BC_OUT5. (C_Y1)
- new net: REG_HL_OUT6. (L_Y1), REG_L6. (Q)
- new net: REG_H5. (Q), REG_HL_OUT5. (L_Y1)
- new net: REG_HL_OUT5. (L_Y1), REG_L5. (Q)
- new net: REG_B3. (Q), REG_BC_OUT3. (C_Y1)
- new net: REG_BC_OUT1. (C_Y1), REG_C1. (Q)
- new net: REG_A0. (Q), REG_A_OUT0. (B_Y)
- new net: REG_DE_OUT1. (D_Y1), REG_E1. (Q)
Changed lines of the file:
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@@
 	(title_block
 		(title "SM83 CPU")
-		(date "2026-03-22")
-		(rev "0.10")
+		(date "2026-04-11")
+		(rev "0.11")
 		(company "CC-BY-SA-4.0 Michael Singer")
 		(comment 1 "https://github.com/msinger/dmg-schematics")
