File: sm83/reg_sp_pc.kicad_sch (KiCad schematic)
At the start: 52 parts

Commit message: SM83: Add schematic of IDU
Parts:
- added unit 2 of REG_PCH_NOT_WE
- added unit 1 of REG_PCL_NOT_WE
Connections:
- net CTL_REG_PC_WE: now also REG_PCL_NOT_WE.1; no longer REG_PCL_NOT_WE.1
- net SYS_RESET: now also REG_PCH_NOT_WE.3; no longer REG_PCH_NOT_WE.3
- new net: REG_PCL0. (~{Q}), REG_PCL1. (~{Q}), REG_PCL2. (~{Q}), REG_PCL3. (~{Q}), REG_PCL4. (~{Q}), REG_PCL5. (~{Q}), REG_PCL6. (~{Q}), REG_PCL7. (~{Q}), REG_PCL_NOT_WE.4
- new net: REG_PCL0. (~{Q}), REG_PCL1. (~{Q}), REG_PCL2. (~{Q}), REG_PCL3. (~{Q}), REG_PCL4. (~{Q}), REG_PCL5. (~{Q}), REG_PCL6. (~{Q}), REG_PCL7. (~{Q}), REG_PCL_NOT_WE.2
- new net: REG_SPL0. (~{Q}), REG_SPL1. (~{Q}), REG_SPL2. (~{Q}), REG_SPL3. (~{Q}), REG_SPL4. (~{Q}), REG_SPL5. (~{Q}), REG_SPL6. (~{Q}), REG_SPL7. (~{Q}), REG_SPL_NOT_WE.2
- new net: REG_SPH0. (~{Q}), REG_SPH1. (~{Q}), REG_SPH2. (~{Q}), REG_SPH3. (~{Q}), REG_SPH4. (~{Q}), REG_SPH5. (~{Q}), REG_SPH6. (~{Q}), REG_SPH7. (~{Q}), REG_SPH_NOT_WE.2
- new net: REG_PCH0. (~{Q}), REG_PCH1. (~{Q}), REG_PCH2. (~{Q}), REG_PCH3. (~{Q}), REG_PCH4. (~{Q}), REG_PCH5. (~{Q}), REG_PCH6. (~{Q}), REG_PCH7. (~{Q}), REG_PCH_NOT_WE.2
- new net: REG_PCH0. (~{Q}), REG_PCH1. (~{Q}), REG_PCH2. (~{Q}), REG_PCH3. (~{Q}), REG_PCH4. (~{Q}), REG_PCH5. (~{Q}), REG_PCH6. (~{Q}), REG_PCH7. (~{Q}), REG_PCH_NOT_WE.4

Commit message: SM83: Add schematic for interrupt handling
Connections:
- new net: REG_PCL0. (~{Q}), REG_PCL1. (~{Q}), REG_PCL2. (~{Q}), REG_PCL3. (~{Q}), REG_PCL4. (~{Q}), REG_PCL5. (~{Q}), REG_PCL6. (~{Q}), REG_PCL7. (~{Q}), REG_PCL_NOT_WE.4
- new net: REG_PCL0. (~{Q}), REG_PCL1. (~{Q}), REG_PCL2. (~{Q}), REG_PCL3. (~{Q}), REG_PCL4. (~{Q}), REG_PCL5. (~{Q}), REG_PCL6. (~{Q}), REG_PCL7. (~{Q}), REG_PCL_NOT_WE.2
- new net: REG_SPL0. (~{Q}), REG_SPL1. (~{Q}), REG_SPL2. (~{Q}), REG_SPL3. (~{Q}), REG_SPL4. (~{Q}), REG_SPL5. (~{Q}), REG_SPL6. (~{Q}), REG_SPL7. (~{Q}), REG_SPL_NOT_WE.2
- new net: REG_SPH0. (~{Q}), REG_SPH1. (~{Q}), REG_SPH2. (~{Q}), REG_SPH3. (~{Q}), REG_SPH4. (~{Q}), REG_SPH5. (~{Q}), REG_SPH6. (~{Q}), REG_SPH7. (~{Q}), REG_SPH_NOT_WE.2
- new net: REG_PCH0. (~{Q}), REG_PCH1. (~{Q}), REG_PCH2. (~{Q}), REG_PCH3. (~{Q}), REG_PCH4. (~{Q}), REG_PCH5. (~{Q}), REG_PCH6. (~{Q}), REG_PCH7. (~{Q}), REG_PCH_NOT_WE.2
- new net: REG_PCH0. (~{Q}), REG_PCH1. (~{Q}), REG_PCH2. (~{Q}), REG_PCH3. (~{Q}), REG_PCH4. (~{Q}), REG_PCH5. (~{Q}), REG_PCH6. (~{Q}), REG_PCH7. (~{Q}), REG_PCH_NOT_WE.4
Changed lines of the file:
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@@
 	(bus
 		(pts
-			(xy 557.53 508) (xy 557.53 533.4)
+			(xy 557.53 508) (xy 557.53 563.88)
 		)
 		(stroke
@@
 		)
 	)
+	(bus
+		(pts
+			(xy 62.23 563.88) (xy 557.53 563.88)
+		)
+		(stroke
+			(width 0)
+			(type default)
+		)
+	)
 	(wire
 		(pts
@@
 		(effects
 			(font
+				(size 1.27 1.27)
+			)
+			(justify right)
+		)
+	)
+	(hierarchical_label "INT_VECTOR[3..7]"
+		(shape input)
+		(at 62.23 563.88 180)
+		(effects
+			(font

Commit message: Finish SM83 CPU schematic
Connections:
- new net: REG_PCL0. (~{Q}), REG_PCL1. (~{Q}), REG_PCL2. (~{Q}), REG_PCL3. (~{Q}), REG_PCL4. (~{Q}), REG_PCL5. (~{Q}), REG_PCL6. (~{Q}), REG_PCL7. (~{Q}), REG_PCL_NOT_WE.4
- new net: REG_PCL0. (~{Q}), REG_PCL1. (~{Q}), REG_PCL2. (~{Q}), REG_PCL3. (~{Q}), REG_PCL4. (~{Q}), REG_PCL5. (~{Q}), REG_PCL6. (~{Q}), REG_PCL7. (~{Q}), REG_PCL_NOT_WE.2
- new net: REG_SPL0. (~{Q}), REG_SPL1. (~{Q}), REG_SPL2. (~{Q}), REG_SPL3. (~{Q}), REG_SPL4. (~{Q}), REG_SPL5. (~{Q}), REG_SPL6. (~{Q}), REG_SPL7. (~{Q}), REG_SPL_NOT_WE.2
- new net: REG_SPH0. (~{Q}), REG_SPH1. (~{Q}), REG_SPH2. (~{Q}), REG_SPH3. (~{Q}), REG_SPH4. (~{Q}), REG_SPH5. (~{Q}), REG_SPH6. (~{Q}), REG_SPH7. (~{Q}), REG_SPH_NOT_WE.2
- new net: REG_PCH0. (~{Q}), REG_PCH1. (~{Q}), REG_PCH2. (~{Q}), REG_PCH3. (~{Q}), REG_PCH4. (~{Q}), REG_PCH5. (~{Q}), REG_PCH6. (~{Q}), REG_PCH7. (~{Q}), REG_PCH_NOT_WE.2
- new net: REG_PCH0. (~{Q}), REG_PCH1. (~{Q}), REG_PCH2. (~{Q}), REG_PCH3. (~{Q}), REG_PCH4. (~{Q}), REG_PCH5. (~{Q}), REG_PCH6. (~{Q}), REG_PCH7. (~{Q}), REG_PCH_NOT_WE.4
Changed lines of the file:
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@@
 	(title_block
 		(title "SM83 CPU")
-		(date "2025-12-08")
+		(date "2025-12-24")
 		(rev "0")
 		(company "CC-BY-SA-4.0 Michael Singer")

Commit message: SM83: Merge dist. NANDs and NOR from IRQ_PRIOs
Connections:
- new net: REG_PCL0. (~{Q}), REG_PCL1. (~{Q}), REG_PCL2. (~{Q}), REG_PCL3. (~{Q}), REG_PCL4. (~{Q}), REG_PCL5. (~{Q}), REG_PCL6. (~{Q}), REG_PCL7. (~{Q}), REG_PCL_NOT_WE.4
- new net: REG_PCL0. (~{Q}), REG_PCL1. (~{Q}), REG_PCL2. (~{Q}), REG_PCL3. (~{Q}), REG_PCL4. (~{Q}), REG_PCL5. (~{Q}), REG_PCL6. (~{Q}), REG_PCL7. (~{Q}), REG_PCL_NOT_WE.2
- new net: REG_SPL0. (~{Q}), REG_SPL1. (~{Q}), REG_SPL2. (~{Q}), REG_SPL3. (~{Q}), REG_SPL4. (~{Q}), REG_SPL5. (~{Q}), REG_SPL6. (~{Q}), REG_SPL7. (~{Q}), REG_SPL_NOT_WE.2
- new net: REG_SPH0. (~{Q}), REG_SPH1. (~{Q}), REG_SPH2. (~{Q}), REG_SPH3. (~{Q}), REG_SPH4. (~{Q}), REG_SPH5. (~{Q}), REG_SPH6. (~{Q}), REG_SPH7. (~{Q}), REG_SPH_NOT_WE.2
- new net: REG_PCH0. (~{Q}), REG_PCH1. (~{Q}), REG_PCH2. (~{Q}), REG_PCH3. (~{Q}), REG_PCH4. (~{Q}), REG_PCH5. (~{Q}), REG_PCH6. (~{Q}), REG_PCH7. (~{Q}), REG_PCH_NOT_WE.2
- new net: REG_PCH0. (~{Q}), REG_PCH1. (~{Q}), REG_PCH2. (~{Q}), REG_PCH3. (~{Q}), REG_PCH4. (~{Q}), REG_PCH5. (~{Q}), REG_PCH6. (~{Q}), REG_PCH7. (~{Q}), REG_PCH_NOT_WE.4
Changed lines of the file:
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@@
 	(title_block
 		(title "SM83 CPU")
-		(date "2025-12-24")
+		(date "2025-12-25")
 		(rev "0")
 		(company "CC-BY-SA-4.0 Michael Singer")

Commit message: Release version 0.9 of both schematics
Connections:
- new net: REG_PCL0. (~{Q}), REG_PCL1. (~{Q}), REG_PCL2. (~{Q}), REG_PCL3. (~{Q}), REG_PCL4. (~{Q}), REG_PCL5. (~{Q}), REG_PCL6. (~{Q}), REG_PCL7. (~{Q}), REG_PCL_NOT_WE.4
- new net: REG_PCL0. (~{Q}), REG_PCL1. (~{Q}), REG_PCL2. (~{Q}), REG_PCL3. (~{Q}), REG_PCL4. (~{Q}), REG_PCL5. (~{Q}), REG_PCL6. (~{Q}), REG_PCL7. (~{Q}), REG_PCL_NOT_WE.2
- new net: REG_SPL0. (~{Q}), REG_SPL1. (~{Q}), REG_SPL2. (~{Q}), REG_SPL3. (~{Q}), REG_SPL4. (~{Q}), REG_SPL5. (~{Q}), REG_SPL6. (~{Q}), REG_SPL7. (~{Q}), REG_SPL_NOT_WE.2
- new net: REG_SPH0. (~{Q}), REG_SPH1. (~{Q}), REG_SPH2. (~{Q}), REG_SPH3. (~{Q}), REG_SPH4. (~{Q}), REG_SPH5. (~{Q}), REG_SPH6. (~{Q}), REG_SPH7. (~{Q}), REG_SPH_NOT_WE.2
- new net: REG_PCH0. (~{Q}), REG_PCH1. (~{Q}), REG_PCH2. (~{Q}), REG_PCH3. (~{Q}), REG_PCH4. (~{Q}), REG_PCH5. (~{Q}), REG_PCH6. (~{Q}), REG_PCH7. (~{Q}), REG_PCH_NOT_WE.2
- new net: REG_PCH0. (~{Q}), REG_PCH1. (~{Q}), REG_PCH2. (~{Q}), REG_PCH3. (~{Q}), REG_PCH4. (~{Q}), REG_PCH5. (~{Q}), REG_PCH6. (~{Q}), REG_PCH7. (~{Q}), REG_PCH_NOT_WE.4
Changed lines of the file:
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@@
 		(title "SM83 CPU")
 		(date "2025-12-25")
-		(rev "0")
+		(rev "0.9")
 		(company "CC-BY-SA-4.0 Michael Singer")
 		(comment 1 "https://github.com/msinger/dmg-schematics")

Commit message: Release revision 0.10 of both schematics
Connections:
- new net: REG_PCL0. (~{Q}), REG_PCL1. (~{Q}), REG_PCL2. (~{Q}), REG_PCL3. (~{Q}), REG_PCL4. (~{Q}), REG_PCL5. (~{Q}), REG_PCL6. (~{Q}), REG_PCL7. (~{Q}), REG_PCL_NOT_WE.4
- new net: REG_PCL0. (~{Q}), REG_PCL1. (~{Q}), REG_PCL2. (~{Q}), REG_PCL3. (~{Q}), REG_PCL4. (~{Q}), REG_PCL5. (~{Q}), REG_PCL6. (~{Q}), REG_PCL7. (~{Q}), REG_PCL_NOT_WE.2
- new net: REG_SPL0. (~{Q}), REG_SPL1. (~{Q}), REG_SPL2. (~{Q}), REG_SPL3. (~{Q}), REG_SPL4. (~{Q}), REG_SPL5. (~{Q}), REG_SPL6. (~{Q}), REG_SPL7. (~{Q}), REG_SPL_NOT_WE.2
- new net: REG_SPH0. (~{Q}), REG_SPH1. (~{Q}), REG_SPH2. (~{Q}), REG_SPH3. (~{Q}), REG_SPH4. (~{Q}), REG_SPH5. (~{Q}), REG_SPH6. (~{Q}), REG_SPH7. (~{Q}), REG_SPH_NOT_WE.2
- new net: REG_PCH0. (~{Q}), REG_PCH1. (~{Q}), REG_PCH2. (~{Q}), REG_PCH3. (~{Q}), REG_PCH4. (~{Q}), REG_PCH5. (~{Q}), REG_PCH6. (~{Q}), REG_PCH7. (~{Q}), REG_PCH_NOT_WE.2
- new net: REG_PCH0. (~{Q}), REG_PCH1. (~{Q}), REG_PCH2. (~{Q}), REG_PCH3. (~{Q}), REG_PCH4. (~{Q}), REG_PCH5. (~{Q}), REG_PCH6. (~{Q}), REG_PCH7. (~{Q}), REG_PCH_NOT_WE.4
Changed lines of the file:
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@@
 	(title_block
 		(title "SM83 CPU")
-		(date "2025-12-25")
-		(rev "0.9")
+		(date "2026-03-22")
+		(rev "0.10")
 		(company "CC-BY-SA-4.0 Michael Singer")
 		(comment 1 "https://github.com/msinger/dmg-schematics")
@@
 		)
 		(instances
-			(project ""
+			(project "sm83"
 				(path "/8717d046-1dfd-46fe-a5f7-4e4d2f07de68/4d4d18fe-a98e-4888-b722-e6c6d1e32861/6f13ac1b-5228-4579-9642-7edf0d7e33e6"
 					(reference "REG_PC_OUT0")
@@
 		)
 		(instances
-			(project ""
+			(project "sm83"
 				(path "/8717d046-1dfd-46fe-a5f7-4e4d2f07de68/4d4d18fe-a98e-4888-b722-e6c6d1e32861/6f13ac1b-5228-4579-9642-7edf0d7e33e6"
 					(reference "REG_PC_OUT3")
@@
 		)
 		(instances
-			(project ""
+			(project "sm83"
 				(path "/8717d046-1dfd-46fe-a5f7-4e4d2f07de68/4d4d18fe-a98e-4888-b722-e6c6d1e32861/6f13ac1b-5228-4579-9642-7edf0d7e33e6"
 					(reference "REG_PC_OUT0")
@@
 		)
 		(instances
-			(project ""
+			(project "sm83"
 				(path "/8717d046-1dfd-46fe-a5f7-4e4d2f07de68/4d4d18fe-a98e-4888-b722-e6c6d1e32861/6f13ac1b-5228-4579-9642-7edf0d7e33e6"
 					(reference "REG_PC_OUT3")
@@
 		)
 		(instances
-			(project ""
+			(project "sm83"
 				(path "/8717d046-1dfd-46fe-a5f7-4e4d2f07de68/4d4d18fe-a98e-4888-b722-e6c6d1e32861/6f13ac1b-5228-4579-9642-7edf0d7e33e6"
 					(reference "REG_SPH0")
@@
 		)
 		(instances
-			(project ""
+			(project "sm83"
 				(path "/8717d046-1dfd-46fe-a5f7-4e4d2f07de68/4d4d18fe-a98e-4888-b722-e6c6d1e32861/6f13ac1b-5228-4579-9642-7edf0d7e33e6"
 					(reference "REG_SPH_NOT_WE")
@@
 		)
 		(instances
-			(project ""
+			(project "sm83"
 				(path "/8717d046-1dfd-46fe-a5f7-4e4d2f07de68/4d4d18fe-a98e-4888-b722-e6c6d1e32861/6f13ac1b-5228-4579-9642-7edf0d7e33e6"
 					(reference "REG_PC_OUT6")
@@
 		)
 		(instances
-			(project ""
+			(project "sm83"
 				(path "/8717d046-1dfd-46fe-a5f7-4e4d2f07de68/4d4d18fe-a98e-4888-b722-e6c6d1e32861/6f13ac1b-5228-4579-9642-7edf0d7e33e6"
 					(reference "REG_PC_OUT6")
@@
 		)
 		(instances
-			(project ""
+			(project "sm83"
 				(path "/8717d046-1dfd-46fe-a5f7-4e4d2f07de68/4d4d18fe-a98e-4888-b722-e6c6d1e32861/6f13ac1b-5228-4579-9642-7edf0d7e33e6"
 					(reference "REG_SP_OUT0")
@@
 		)
 		(instances
-			(project ""
+			(project "sm83"
 				(path "/8717d046-1dfd-46fe-a5f7-4e4d2f07de68/4d4d18fe-a98e-4888-b722-e6c6d1e32861/6f13ac1b-5228-4579-9642-7edf0d7e33e6"
 					(reference "REG_PC_OUT0")
@@
 		)
 		(instances
-			(project ""
+			(project "sm83"
 				(path "/8717d046-1dfd-46fe-a5f7-4e4d2f07de68/4d4d18fe-a98e-4888-b722-e6c6d1e32861/6f13ac1b-5228-4579-9642-7edf0d7e33e6"
 					(reference "REG_SP_OUT0")
@@
 		)
 		(instances
-			(project ""
+			(project "sm83"
 				(path "/8717d046-1dfd-46fe-a5f7-4e4d2f07de68/4d4d18fe-a98e-4888-b722-e6c6d1e32861/6f13ac1b-5228-4579-9642-7edf0d7e33e6"
 					(reference "REG_SP_OUT0")
@@
 		)
 		(instances
-			(project ""
+			(project "sm83"
 				(path "/8717d046-1dfd-46fe-a5f7-4e4d2f07de68/4d4d18fe-a98e-4888-b722-e6c6d1e32861/6f13ac1b-5228-4579-9642-7edf0d7e33e6"
 					(reference "REG_PC_OUT6")
@@
 		)
 		(instances
-			(project ""
+			(project "sm83"
 				(path "/8717d046-1dfd-46fe-a5f7-4e4d2f07de68/4d4d18fe-a98e-4888-b722-e6c6d1e32861/6f13ac1b-5228-4579-9642-7edf0d7e33e6"
 					(reference "REG_PC_OUT3")
@@
 		)
 		(instances
-			(project ""
+			(project "sm83"
 				(path "/8717d046-1dfd-46fe-a5f7-4e4d2f07de68/4d4d18fe-a98e-4888-b722-e6c6d1e32861/6f13ac1b-5228-4579-9642-7edf0d7e33e6"
 					(reference "REG_PCH_NOT_WE")
@@
 		)
 		(instances
-			(project ""
+			(project "sm83"
 				(path "/8717d046-1dfd-46fe-a5f7-4e4d2f07de68/4d4d18fe-a98e-4888-b722-e6c6d1e32861/6f13ac1b-5228-4579-9642-7edf0d7e33e6"
 					(reference "REG_PCH_NOT_WE")
@@
 		)
 		(instances
-			(project ""
+			(project "sm83"
 				(path "/8717d046-1dfd-46fe-a5f7-4e4d2f07de68/4d4d18fe-a98e-4888-b722-e6c6d1e32861/6f13ac1b-5228-4579-9642-7edf0d7e33e6"
 					(reference "REG_PCH0")

Commit message: Release revision 0.11 of both schematics
Connections:
- new net: REG_PCL0. (~{Q}), REG_PCL1. (~{Q}), REG_PCL2. (~{Q}), REG_PCL3. (~{Q}), REG_PCL4. (~{Q}), REG_PCL5. (~{Q}), REG_PCL6. (~{Q}), REG_PCL7. (~{Q}), REG_PCL_NOT_WE.4
- new net: REG_PCL0. (~{Q}), REG_PCL1. (~{Q}), REG_PCL2. (~{Q}), REG_PCL3. (~{Q}), REG_PCL4. (~{Q}), REG_PCL5. (~{Q}), REG_PCL6. (~{Q}), REG_PCL7. (~{Q}), REG_PCL_NOT_WE.2
- new net: REG_SPL0. (~{Q}), REG_SPL1. (~{Q}), REG_SPL2. (~{Q}), REG_SPL3. (~{Q}), REG_SPL4. (~{Q}), REG_SPL5. (~{Q}), REG_SPL6. (~{Q}), REG_SPL7. (~{Q}), REG_SPL_NOT_WE.2
- new net: REG_SPH0. (~{Q}), REG_SPH1. (~{Q}), REG_SPH2. (~{Q}), REG_SPH3. (~{Q}), REG_SPH4. (~{Q}), REG_SPH5. (~{Q}), REG_SPH6. (~{Q}), REG_SPH7. (~{Q}), REG_SPH_NOT_WE.2
- new net: REG_PCH0. (~{Q}), REG_PCH1. (~{Q}), REG_PCH2. (~{Q}), REG_PCH3. (~{Q}), REG_PCH4. (~{Q}), REG_PCH5. (~{Q}), REG_PCH6. (~{Q}), REG_PCH7. (~{Q}), REG_PCH_NOT_WE.2
- new net: REG_PCH0. (~{Q}), REG_PCH1. (~{Q}), REG_PCH2. (~{Q}), REG_PCH3. (~{Q}), REG_PCH4. (~{Q}), REG_PCH5. (~{Q}), REG_PCH6. (~{Q}), REG_PCH7. (~{Q}), REG_PCH_NOT_WE.4
Changed lines of the file:
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@@
 	(title_block
 		(title "SM83 CPU")
-		(date "2026-03-22")
-		(rev "0.10")
+		(date "2026-04-11")
+		(rev "0.11")
 		(company "CC-BY-SA-4.0 Michael Singer")
 		(comment 1 "https://github.com/msinger/dmg-schematics")
