File: sm83/reg_wz.kicad_sch (KiCad schematic)
At the start: 43 parts

Commit message: Finish SM83 CPU schematic
Connections:
- new net: REG_W0. (~{Q}), REG_W1. (~{Q}), REG_W2. (~{Q}), REG_W3. (~{Q}), REG_W4. (~{Q}), REG_W5. (~{Q}), REG_W6. (~{Q}), REG_W7. (~{Q}), REG_W_NOT_WE.2
- new net: REG_Z0. (~{Q}), REG_Z1. (~{Q}), REG_Z2. (~{Q}), REG_Z3. (~{Q}), REG_Z4. (~{Q}), REG_Z5. (~{Q}), REG_Z6. (~{Q}), REG_Z7. (~{Q}), REG_Z_NOT_WE.2
Changed lines of the file:
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@@
 	(title_block
 		(title "SM83 CPU")
-		(date "2025-12-08")
+		(date "2025-12-24")
 		(rev "0")
 		(company "CC-BY-SA-4.0 Michael Singer")

Commit message: SM83: Merge dist. NANDs and NOR from IRQ_PRIOs
Connections:
- new net: REG_W0. (~{Q}), REG_W1. (~{Q}), REG_W2. (~{Q}), REG_W3. (~{Q}), REG_W4. (~{Q}), REG_W5. (~{Q}), REG_W6. (~{Q}), REG_W7. (~{Q}), REG_W_NOT_WE.2
- new net: REG_Z0. (~{Q}), REG_Z1. (~{Q}), REG_Z2. (~{Q}), REG_Z3. (~{Q}), REG_Z4. (~{Q}), REG_Z5. (~{Q}), REG_Z6. (~{Q}), REG_Z7. (~{Q}), REG_Z_NOT_WE.2
Changed lines of the file:
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@@
 	(title_block
 		(title "SM83 CPU")
-		(date "2025-12-24")
+		(date "2025-12-25")
 		(rev "0")
 		(company "CC-BY-SA-4.0 Michael Singer")

Commit message: Release version 0.9 of both schematics
Connections:
- new net: REG_W0. (~{Q}), REG_W1. (~{Q}), REG_W2. (~{Q}), REG_W3. (~{Q}), REG_W4. (~{Q}), REG_W5. (~{Q}), REG_W6. (~{Q}), REG_W7. (~{Q}), REG_W_NOT_WE.2
- new net: REG_Z0. (~{Q}), REG_Z1. (~{Q}), REG_Z2. (~{Q}), REG_Z3. (~{Q}), REG_Z4. (~{Q}), REG_Z5. (~{Q}), REG_Z6. (~{Q}), REG_Z7. (~{Q}), REG_Z_NOT_WE.2
Changed lines of the file:
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@@
 		(title "SM83 CPU")
 		(date "2025-12-25")
-		(rev "0")
+		(rev "0.9")
 		(company "CC-BY-SA-4.0 Michael Singer")
 		(comment 1 "https://github.com/msinger/dmg-schematics")

Commit message: Release revision 0.10 of both schematics
Connections:
- new net: REG_W0. (~{Q}), REG_W1. (~{Q}), REG_W2. (~{Q}), REG_W3. (~{Q}), REG_W4. (~{Q}), REG_W5. (~{Q}), REG_W6. (~{Q}), REG_W7. (~{Q}), REG_W_NOT_WE.2
- new net: REG_Z0. (~{Q}), REG_Z1. (~{Q}), REG_Z2. (~{Q}), REG_Z3. (~{Q}), REG_Z4. (~{Q}), REG_Z5. (~{Q}), REG_Z6. (~{Q}), REG_Z7. (~{Q}), REG_Z_NOT_WE.2
Changed lines of the file:
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@@
 	(title_block
 		(title "SM83 CPU")
-		(date "2025-12-25")
-		(rev "0.9")
+		(date "2026-03-22")
+		(rev "0.10")
 		(company "CC-BY-SA-4.0 Michael Singer")
 		(comment 1 "https://github.com/msinger/dmg-schematics")
@@
 		)
 		(instances
-			(project ""
+			(project "sm83"
 				(path "/8717d046-1dfd-46fe-a5f7-4e4d2f07de68/4d4d18fe-a98e-4888-b722-e6c6d1e32861/2d896e4f-a722-4032-a79a-2d52cd584a24"
 					(reference "REG_NOT0")
@@
 		)
 		(instances
-			(project ""
+			(project "sm83"
 				(path "/8717d046-1dfd-46fe-a5f7-4e4d2f07de68/4d4d18fe-a98e-4888-b722-e6c6d1e32861/2d896e4f-a722-4032-a79a-2d52cd584a24"
 					(reference "REG_W0")
@@
 		)
 		(instances
-			(project ""
+			(project "sm83"
 				(path "/8717d046-1dfd-46fe-a5f7-4e4d2f07de68/4d4d18fe-a98e-4888-b722-e6c6d1e32861/2d896e4f-a722-4032-a79a-2d52cd584a24"
 					(reference "REG_WZ_OUT0")
@@
 		)
 		(instances
-			(project ""
+			(project "sm83"
 				(path "/8717d046-1dfd-46fe-a5f7-4e4d2f07de68/4d4d18fe-a98e-4888-b722-e6c6d1e32861/2d896e4f-a722-4032-a79a-2d52cd584a24"
 					(reference "REG_W_NOT_WE")
@@
 		)
 		(instances
-			(project ""
+			(project "sm83"
 				(path "/8717d046-1dfd-46fe-a5f7-4e4d2f07de68/4d4d18fe-a98e-4888-b722-e6c6d1e32861/2d896e4f-a722-4032-a79a-2d52cd584a24"
 					(reference "REG_OR")
@@
 		)
 		(instances
-			(project ""
+			(project "sm83"
 				(path "/8717d046-1dfd-46fe-a5f7-4e4d2f07de68/4d4d18fe-a98e-4888-b722-e6c6d1e32861/2d896e4f-a722-4032-a79a-2d52cd584a24"
 					(reference "REG_BUS_PCH_B0")

Commit message: Release revision 0.11 of both schematics
Connections:
- new net: REG_W0. (~{Q}), REG_W1. (~{Q}), REG_W2. (~{Q}), REG_W3. (~{Q}), REG_W4. (~{Q}), REG_W5. (~{Q}), REG_W6. (~{Q}), REG_W7. (~{Q}), REG_W_NOT_WE.2
- new net: REG_Z0. (~{Q}), REG_Z1. (~{Q}), REG_Z2. (~{Q}), REG_Z3. (~{Q}), REG_Z4. (~{Q}), REG_Z5. (~{Q}), REG_Z6. (~{Q}), REG_Z7. (~{Q}), REG_Z_NOT_WE.2
Changed lines of the file:
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@@
 	(title_block
 		(title "SM83 CPU")
-		(date "2026-03-22")
-		(rev "0.10")
+		(date "2026-04-11")
+		(rev "0.11")
 		(company "CC-BY-SA-4.0 Michael Singer")
 		(comment 1 "https://github.com/msinger/dmg-schematics")
