File: dmg_cpu_b/sprite_store_part1.kicad_sch (KiCad schematic)
At the start: 100 parts

Commit message: Give more meaningful names to cell types
Before this commit, many of the cells types in the chip were named in a
sloppy manner. The different inverter, latch and flip flop valiants were
just suffixed with A, B, C, D, ... Those suffixes gave no information
about the actual differences. They had to be looked up in the
documentation. Now the names of cell types with different variants have
changed:

* Inverter types are named NOT_X1, NOT_X2, NOT_X3, ... The _Xn suffix
  reflects the drive strength of the cell. X1 is the drive strength of
  the weakest inverter, X2 is double the drive strength of the weakest
  inverter.
* Flip flop types are named DFFR, DFFR_CC, DFFR_CC_Q. DFFR is a normal
  data flip flop with reset and a single clock input. The suffix _CC is
  added to flip flops that have two complementary clock inputs (CLK and
  /CLK). Flip flops that only have the positive Q output are suffixed
  with _Q.
* Latch types are named similar to flip flops: DLATCH, DLATCH_EE,
  DLATCH_EE_Q. The suffix _EE is given to latches that require
  "externally inverted enable" signals (ENA and /ENA).
* I/O pad types all start with PAD_BIDIR, PAD_IN or PAD_OUT. They also
  have suffixes that describe what makes them unique, like _PU for
  pull-ups.

Other minor changes were made to align the names with common naming
schemes of other cell libraries.
Parts:
- ABOP, ABUG, AMES, AROF, BECA, BOXA, BOZU, BUHE, BULU, BUNA, BYHU, CADU, CAJU, CAJY, CAPO, CEBO, COMA, CONO, CUFA, CUFO, CUMU, CUZA, DAFU, DEBA, DESE, DEVY, DUHA, DUNY, FYHY, GYHO, WANU, WYTE, XABO, XAVE, XAZY, XEFE, XEGE, XOSY, XYNU, YGUS, YKUK, YLOV, YSOK, YWAK, YZEP, ZENE, ZONY, ZURO, ZURY, ZYLU: value D_LATCH_A -> DLATCH_EE; symbol DMG_CPU_Cells:D_LATCH_A -> DMG_CPU_Cells:DLATCH_EE
- AFOZ, AHUM, AJAL, APON, AXEC, BACO, BEFE, BEMO, BETY, BEVY, BOVE, BUCE, BUKY, BYDO, BYRO, CEGY, CELU, CUBE, CUBO, CUVU, CYBY, CYRO, DEZU, DONY, DOWA, DYGO, EFUD, ENAP, GOFO, WAJA, WEHE, WEPY, WERE, WERU, WOKO, WOXY, WUXE, WUXU, XYRE, YJEM, YWAV, ZABY, ZAVE, ZECE, ZEDY, ZETU, ZEXE, ZUKE, ZUMU, ZYPO: value TRI_INV_IF0 -> NOT_IF0; symbol DMG_CPU_Cells:TRI_INV_IF0 -> DMG_CPU_Cells:NOT_IF0
